Commit message: Merge into one superfunction for fitting. Includes joint limit constraints. Also improve joint limits on fingertips

File: software/control/src/urdf/robotiq_simple_collision.urdf (robot description, URDF)
Before this commit: robot s-model_articulated, 13 links, 12 joints
Joints:
- joint finger_1_joint_2: limit lower=-0.7854 upper=3.1416 effort=100 velocity=100 -> lower=-0.7854 upper=0.7854 effort=100 velocity=100
- joint finger_2_joint_2: limit lower=-0.7854 upper=3.1416 effort=100 velocity=100 -> lower=-0.7854 upper=0.7854 effort=100 velocity=100
- joint finger_middle_joint_2: limit lower=-0.7854 upper=3.1416 effort=100 velocity=100 -> lower=-0.7854 upper=0.7854 effort=100 velocity=100
