Commit message: Bind joints in lower fingers for now

File: software/control/src/urdf/irb140_chull_robotiq.urdf (robot description, URDF)
Before this commit: robot IRB140_-_M2004C_Complete_base.SLDASM, 21 links, 20 joints
Joints:
- joint left_finger_1_joint_1: limit lower=0 upper=1.5708 effort=100 velocity=100 -> lower=0 upper=0 effort=100 velocity=100
- joint left_finger_1_joint_2: limit lower=-0.7854 upper=0.7854 effort=100 velocity=100 -> lower=-0.7854 upper=-0.7854 effort=100 velocity=100
- joint left_finger_2_joint_1: limit lower=0 upper=1.5708 effort=100 velocity=100 -> lower=0 upper=0 effort=100 velocity=100
- joint left_finger_2_joint_2: limit lower=-0.7854 upper=0.7854 effort=100 velocity=100 -> lower=-0.7854 upper=-0.7854 effort=100 velocity=100
- joint left_finger_middle_joint_1: limit lower=0 upper=1.5708 effort=100 velocity=100 -> lower=0 upper=0 effort=100 velocity=100
- joint left_finger_middle_joint_2: limit lower=-0.7854 upper=0.7854 effort=100 velocity=100 -> lower=-0.7854 upper=-0.7854 effort=100 velocity=100
