Commit message: Better cardboard box model

File: software/control/src/urdf/cardbox_box_hollow_with_lid.urdf (robot description, URDF)
Before this commit: robot cardboard_box, 9 links, 8 joints
Links:
- link box_lid_nx: geometry collision box size=0.125 0.27 0.005; visual box size=0.125 0.27 0.005
- link box_lid_ny: geometry collision box size=0.345 0.125 0.005; visual box size=0.345 0.125 0.005
- link box_lid_px: geometry collision box size=0.125 0.27 0.005; visual box size=0.125 0.27 0.005
- link box_lid_py: geometry collision box size=0.345 0.125 0.005; visual box size=0.345 0.125 0.005
