Commit message: Remove PCL dependency, get finger state piped in

File: software/control/src/urdf/irb140_chull_robotiq_actuated_fingers.urdf (robot description, URDF)
Before this commit: robot IRB140_-_M2004C_Complete_base.SLDASM, 21 links, 20 joints
Joints:
- removed joint left_finger_1_joint_0
- removed joint left_finger_2_joint_0
- removed joint left_finger_middle_joint_0
- added joint left_finger_1_joint_3: type revolute, parent finger_1_link_2, child finger_1_link_3, origin xyz=0.039 0 0 rpy=0 0 0, axis 0 0 1, limit lower=0 upper=3.1416 effort=100 velocity=100
- added joint left_finger_2_joint_3: type revolute, parent finger_2_link_2, child finger_2_link_3, origin xyz=0.039 0 0 rpy=0 0 0, axis 0 0 1, limit lower=-1.57 upper=3.14 effort=100 velocity=100
- added joint left_finger_middle_joint_3: type revolute, parent finger_middle_link_2, child finger_middle_link_3, origin xyz=0.039 0 0 rpy=0 0 0, axis 0 0 1, limit lower=-1.57 upper=3.14 effort=100 velocity=100
- joint left_finger_1_joint_1: child finger_1_link_2 -> finger_1_link_1; limit lower=0 upper=1.57 effort=100 velocity=100 -> lower=0 upper=3.1416 effort=100 velocity=100; origin xyz=0.050 -.028 0 rpy=0 0 -0.52 -> xyz=0.020 0 0 rpy=0 0 0; parent finger_1_link_1 -> finger_1_link_0
- joint left_finger_1_joint_2: child finger_1_link_3 -> finger_1_link_2; limit lower=-0.7854 upper=3.14 effort=100 velocity=100 -> lower=0 upper=3.1416 effort=100 velocity=100; origin xyz=0.039 0 0 rpy=0 0 0 -> xyz=0.050 -.028 0 rpy=0 0 -0.52; parent finger_1_link_2 -> finger_1_link_1
- joint left_finger_2_joint_1: child finger_2_link_2 -> finger_2_link_1; limit lower=0 upper=1.57 effort=100 velocity=100 -> lower=-0.5 upper=2.0 effort=100 velocity=100; origin xyz=0.050 -.028 0 rpy=0 0 -0.52 -> xyz=0.020 0 0 rpy=0 0 0; parent finger_2_link_1 -> finger_2_link_0
- joint left_finger_2_joint_2: child finger_2_link_3 -> finger_2_link_2; limit lower=-0.7854 upper=3.14 effort=100 velocity=100 -> lower=-1.57 upper=3.14 effort=100 velocity=100; origin xyz=0.039 0 0 rpy=0 0 0 -> xyz=0.050 -.028 0 rpy=0 0 -0.52; parent finger_2_link_2 -> finger_2_link_1
- joint left_finger_middle_joint_1: child finger_middle_link_2 -> finger_middle_link_1; limit lower=0 upper=1.57 effort=100 velocity=100 -> lower=-0.5 upper=2.0 effort=100 velocity=100; origin xyz=0.050 -.028 0 rpy=0 0 -0.52 -> xyz=0.020 0 0 rpy=0 0 0; parent finger_middle_link_1 -> finger_middle_link_0
- joint left_finger_middle_joint_2: child finger_middle_link_3 -> finger_middle_link_2; limit lower=-0.7854 upper=3.14 effort=100 velocity=100 -> lower=-1.57 upper=3.14 effort=100 velocity=100; origin xyz=0.039 0 0 rpy=0 0 0 -> xyz=0.050 -.028 0 rpy=0 0 -0.52; parent finger_middle_link_2 -> finger_middle_link_1
