Commit message: Lots of development on DART replication

File: software/control/src/jasmine_tea_box.urdf (robot description, URDF)
Before this commit: robot compressed_air_can, 2 links, 0 joints
Links:
- removed link cylinder
- added link box, mass 0.5; collision box size=0.14 0.07 0.225; visual box size=0.14 0.07 0.225

Commit message: Sort of works with full IRB plus hand on dynamic data. Cool! But slow.

File: software/control/src/jasmine_tea_box.urdf (robot description, URDF)
Before this commit: robot jasmine_tea_box, 2 links, 0 joints
Links:
- link desk: geometry collision box size=0.5 0.75 0.05; visual box size=0.3 0.3 0.05

Commit message: Better tuning, downsampling, better gain derivation

File: software/control/src/jasmine_tea_box.urdf (robot description, URDF)
Before this commit: robot jasmine_tea_box, 2 links, 0 joints
Links:
- link desk: geometry collision box size=0.5 0.75 0.05; visual box size=0.5 0.75 0.05

File: software/control/src/urdf/irb140_chull_robotiq.urdf (robot description, URDF)
Before this commit: robot IRB140_-_M2004C_Complete_base.SLDASM, 21 links, 20 joints
Joints:
- removed joint finger_1_joint_0
- removed joint finger_1_joint_1
- removed joint finger_1_joint_2
- removed joint finger_2_joint_0
- removed joint finger_2_joint_1
- removed joint finger_2_joint_2
- removed joint finger_middle_joint_0
- removed joint finger_middle_joint_1
- removed joint finger_middle_joint_2
- removed joint palm_finger_1_joint
- removed joint palm_finger_2_joint
- removed joint palm_finger_middle_joint
- added joint left_finger_1_joint_0: type revolute, parent finger_1_link_0, child finger_1_link_1, origin xyz=0.020 0 0 rpy=0 0 0, axis 0 0 1, limit lower=0 upper=1.055 effort=100 velocity=100
- added joint left_finger_1_joint_1: type revolute, parent finger_1_link_1, child finger_1_link_2, origin xyz=0.050 -.028 0 rpy=0 0 -0.52, axis 0 0 1, limit lower=0 upper=1.5708 effort=100 velocity=100
- added joint left_finger_1_joint_2: type revolute, parent finger_1_link_2, child finger_1_link_3, origin xyz=0.039 0 0 rpy=0 0 0, axis 0 0 1, limit lower=-0.7854 upper=0.7854 effort=100 velocity=100
- added joint left_finger_2_joint_0: type revolute, parent finger_2_link_0, child finger_2_link_1, origin xyz=0.020 0 0 rpy=0 0 0, axis 0 0 1, limit lower=0 upper=1.055 effort=100 velocity=100
- added joint left_finger_2_joint_1: type revolute, parent finger_2_link_1, child finger_2_link_2, origin xyz=0.050 -.028 0 rpy=0 0 -0.52, axis 0 0 1, limit lower=0 upper=1.5708 effort=100 velocity=100
- added joint left_finger_2_joint_2: type revolute, parent finger_2_link_2, child finger_2_link_3, origin xyz=0.039 0 0 rpy=0 0 0, axis 0 0 1, limit lower=-0.7854 upper=0.7854 effort=100 velocity=100
- added joint left_finger_middle_joint_0: type revolute, parent finger_middle_link_0, child finger_middle_link_1, origin xyz=0.020 0 0 rpy=0 0 0, axis 0 0 1, limit lower=0 upper=1.055 effort=100 velocity=100
- added joint left_finger_middle_joint_1: type revolute, parent finger_middle_link_1, child finger_middle_link_2, origin xyz=0.050 -.028 0 rpy=0 0 -0.52, axis 0 0 1, limit lower=0 upper=1.5708 effort=100 velocity=100
- added joint left_finger_middle_joint_2: type revolute, parent finger_middle_link_2, child finger_middle_link_3, origin xyz=0.039 0 0 rpy=0 0 0, axis 0 0 1, limit lower=-0.7854 upper=0.7854 effort=100 velocity=100
- added joint left_palm_finger_1_joint: type fixed, parent palm, child finger_1_link_0, origin xyz=-0.0455 0.0214 0.036 rpy=0 3.1416 -1.57, axis 0 1 0
- added joint left_palm_finger_2_joint: type fixed, parent palm, child finger_2_link_0, origin xyz=-0.0455 0.0214 -0.036 rpy=0 3.1416 -1.57, axis 0 1 0
- added joint left_palm_finger_middle_joint: type fixed, parent palm, child finger_middle_link_0, origin xyz=0.0455 0.0214 0 rpy=0 0 1.57, axis 0 0 1
