Commit message: Prep for director integration with estimator

File: software/control/src/desk.urdf (robot description, URDF)
Before this commit: robot jasmine_tea_box, 1 links, 0 joints
Links:
- removed link box
- added link desk, mass 0.5; collision box size=0.5 0.75 0.05; visual box size=0.5 0.75 0.05

Commit message: Fix free  space constraints, fix some run rate bugs

File: software/control/src/desk.urdf (robot description, URDF)
Before this commit: robot desk, 1 links, 0 joints
Links:
- link desk: geometry collision box size=0.5 0.75 0.5; visual box size=0.5 0.75 0.5
