Commit message: Finger mounts properly attached for wsg50 urdf

File: software/models/common_components/schunk_description/urdf/wsg/wsg_50.urdf (robot description, URDF)
Before this commit: robot wsg_50, 3 links, 2 joints
Joints:
- joint wsg_50_finger_left_joint: origin xyz=0 0 0.0789 rpy=0 0 0 -> xyz=0 -0.0719 0 rpy=3.1415 3.1415 0
- joint wsg_50_finger_right_joint: origin xyz=0 0 0.0789 rpy=-0 0 0 -> xyz=0 -0.0719 0.0 rpy=3.1415 0 0

File: software/models/common_components/schunk_description/urdf/wsg/wsg_50.urdf.xacro (robot description, xacro)
@@ -10,15 +10,15 @@
     <visual>
       <geometry>
-        <mesh filename="package://schunk_description/meshes/wsg_50/palm.stl" />
+        <mesh filename="package://schunk_description/meshes/wsg_50/palm.stl"/>
       </geometry>
     </visual>
     <collision>
       <geometry>
-        <mesh filename="package://schunk_description/meshes/wsg_50/palm.stl" />
+        <mesh filename="package://schunk_description/meshes/wsg_50/palm.stl"/>
       </geometry>
     </collision>
   </link>
   <joint name="${name}_finger_left_joint" type="prismatic" >
-    <origin xyz="0 0 0.0789" rpy="0 0 0"/>
+    <origin xyz="0 -0.0719 0" rpy="3.1415 3.1415 0"/>
     <parent link="${name}_palm_link" />
     <child link="${name}_finger_left_link" />
@@ -34,15 +34,15 @@
     <visual>
       <geometry>
-        <mesh filename="package://schunk_description/meshes/wsg_50/finger.stl" />
+        <mesh filename="package://schunk_description/meshes/wsg_50/finger.stl"/>
       </geometry>
     </visual>
     <collision>
       <geometry>
-        <mesh filename="package://schunk_description/meshes/wsg_50/finger.stl" />
+        <mesh filename="package://schunk_description/meshes/wsg_50/finger.stl"/>
       </geometry>
     </collision>
   </link>
   <joint name="${name}_finger_right_joint" type="prismatic" >
-    <origin xyz="0 0 0.0789" rpy="-0 0 0"/>
+    <origin xyz="0 -0.0719 0.0" rpy="3.1415 0 0"/>
     <parent link="${name}_palm_link" />
     <child link="${name}_finger_right_link" />
@@ -59,10 +59,10 @@
     <visual>
       <geometry>
-        <mesh filename="package://schunk_description/meshes/wsg_50/finger.stl" />
+        <mesh filename="package://schunk_description/meshes/wsg_50/finger.stl"/>
       </geometry>
     </visual>
     <collision>
       <geometry>
-        <mesh filename="package://schunk_description/meshes/wsg_50/finger.stl" />
+        <mesh filename="package://schunk_description/meshes/wsg_50/finger.stl"/>
       </geometry>
     </collision>
