Commit message: Director loaded in with new hand and reasonable collision meshes for all save thegripper box itself

File: software/models/common_components/schunk_description/urdf/wsg/body.xacro (robot description, xacro)
@@ -1,6 +1,3 @@
-<?xml version="1.0"?>
-<robot xmlns:xacro="http://www.ros.org/wiki/xacro" name="wsg_50">
-  <xacro:include filename="$(find schunk_description)/urdf/wsg/visual_collisions.xacro" />
-  <link name="palm">
+<link name="wsg_50_palm_link">
     <inertial>
       <origin xyz="0 0 0" rpy="0 0 0"/>
@@ -21,8 +18,8 @@
   <joint name="wsg_50_finger_left_joint" type="prismatic" >
     <origin xyz="0 -0.0719 0" rpy="0 1.57 0"/>
-    <parent link="palm" />
+    <parent link="wsg_50_palm_link" />
     <child link="wsg_50_finger_left_link" />
-    <axis xyz="0 0 -1" />
-    <!--<limit effort="10" lower="-0.001" upper="0.109" velocity="1.0"/>-->
+    <axis xyz="0 1 0" />
+    <limit effort="10" lower="-0.001" upper="0.061" velocity="2.0"/>
   </joint>
   <link name="wsg_50_finger_left_link">
@@ -32,14 +29,22 @@
       <inertia ixx="0.01" ixy="0" ixz="0" iyy="0.01" iyz="0" izz="0.01" />
     </inertial>
-    <!-- <xacro:left_finger_simple_visual/> -->
-    <xacro:left_finger_pretty_visual/>
-    <xacro:left_finger_simple_collision/>
+    <visual>
+      <geometry>
+        <mesh filename="package://schunk_description/meshes/wsg_50/finger_without_gelsight.stl"/>
+      </geometry>
+    </visual>
+    <collision>
+      <geometry>
+        <mesh filename="package://schunk_description/meshes/wsg_50/finger_without_gelsight.stl"/>
+      </geometry>
+    </collision>
   </link>
   <joint name="wsg_50_finger_right_joint" type="prismatic" >
     <origin xyz="0 -0.0719 0.0" rpy="3.1415 -1.57 0"/>
-    <parent link="palm" />
+    <parent link="wsg_50_palm_link" />
     <child link="wsg_50_finger_right_link" />
-    <axis xyz="0 0 1" />
-    <!--<limit effort="10" lower="-0.001" upper="0.109" velocity="1.0"/> -->
+    <axis xyz="0 -1 0" />
+    <mimic joint="wsg_50_finger_left_joint" multiplier="1" offset="0"/>
+    <limit effort="10" lower="-0.001" upper="0.061" velocity="2.0"/>
   </joint>
   <link name="wsg_50_finger_right_link">
@@ -49,7 +54,14 @@
       <inertia ixx="0.01" ixy="0" ixz="0" iyy="0.01" iyz="0" izz="0.01" />
     </inertial>
-    <!-- <xacro:right_finger_simple_visual/> -->
-    <xacro:right_finger_pretty_visual/>
-    <xacro:right_finger_simple_collision/>
+    <visual>
+      <geometry>
+        <mesh filename="package://schunk_description/meshes/wsg_50/finger_with_gelsight.stl"/>
+      </geometry>
+    </visual>
+    <collision>
+      <geometry>
+        <mesh filename="package://schunk_description/meshes/wsg_50/finger_with_gelsight.stl"/>
+      </geometry>
+    </collision>
   </link>
   <!-- extensions -->
@@ -70,3 +82,2 @@
     </actuator>
   </transmission>
-</robot>

File: software/models/common_components/schunk_description/urdf/wsg/wsg_50.urdf (robot description, URDF)
Before this commit: robot wsg_50, 3 links, 2 joints
Links:
- removed link wsg_50_palm_link
- added link palm, mass 1; collision mesh filename=package://schunk_description/meshes/wsg_50/palm.stl; visual mesh filename=package://schunk_description/meshes/wsg_50/palm.stl
- link wsg_50_finger_left_link: geometry collision box size=0.0365 0.117 0.0122; visual box size=0.0365 0.117 0.0122
- link wsg_50_finger_right_link: geometry collision box size=0.03 0.0344 0.0344; collision box size=0.0318 0.0318 0.02472
Joints:
- joint wsg_50_finger_left_joint: axis 0 1 0 -> 0 0 -1; limit lower=-0.001 upper=0.061 effort=10 velocity=2.0 -> (none); origin xyz=0 -0.0719 0 rpy=3.1415 3.1415 0 -> xyz=0 -0.0719 0 rpy=0 1.57 0; parent wsg_50_palm_link -> palm
- joint wsg_50_finger_right_joint: axis 0 -1 0 -> 0 0 1; limit lower=-0.001 upper=0.061 effort=10 velocity=2.0 -> (none); mimic joint=wsg_50_finger_left_joint multiplier=1 offset=0 -> (none); origin xyz=0 -0.0719 0.0 rpy=3.1415 0 0 -> xyz=0 -0.0719 0.0 rpy=3.1415 -1.57 0; parent wsg_50_palm_link -> palm
