Commit message: Rough working state for gelsight + kinect tracking

File: software/models/common_components/schunk_description/urdf/wsg/visual_collisions.xacro (robot description, xacro)
@@ -35,8 +35,37 @@
     </collision>
   </xacro:macro>
+  <xacro:macro name="palm_pretty_visual" params="">
+    <visual>
+      <geometry>
+        <mesh filename="package://schunk_description/meshes/wsg_50/palm.stl"/>
+      </geometry>
+    </visual>
+  </xacro:macro>
+  <xacro:macro name="palm_pretty_collision" params="">
+    <collision>
+      <geometry>
+        <mesh filename="package://schunk_description/meshes/wsg_50/palm.stl"/>
+      </geometry>
+    </collision>
+  </xacro:macro>
+  <xacro:macro name="palm_simple_visual" params="">
+    <!-- The gripper itself -->
+    <xacro:visual_offset_box s_x="0.1453" s_y="0.0725" s_z="0.049" o_x="0.00" o_y="-0.0351" o_z="0.0"/>
+    <!-- the larger mounting plate -->
+    <xacro:visual_offset_box s_x="0.05" s_y="0.0064" s_z="0.095" o_x="0.00" o_y="0.007" o_z="0"/>
+  </xacro:macro>
+  <xacro:macro name="palm_simple_collision" params="">
+    <!-- The gripper itself -->
+    <xacro:collision_offset_box s_x="0.1453" s_y="0.0725" s_z="0.049" o_x="0.00" o_y="-0.0351" o_z="0.0"/>
+    <!-- the larger mounting plate -->
+    <xacro:collision_offset_box s_x="0.05" s_y="0.0064" s_z="0.095" o_x="0.00" o_y="0.007" o_z="0"/>
+  </xacro:macro>
   <xacro:macro name="left_finger_pretty_visual" params="">
     <visual>
       <geometry>
         <mesh filename="package://schunk_description/meshes/wsg_50/finger_without_gelsight.stl"/>
+        <material name="mostly_transparent">
+          <color rgb="255 255 255" alpha="0.1"/>
+        </material>
       </geometry>
     </visual>

File: software/models/common_components/schunk_description/urdf/wsg/wsg_50.urdf (robot description, URDF)
Before this commit: robot wsg_50, 3 links, 2 joints
Links:
- link palm: geometry collision box size=0.05 0.0064 0.095; collision box size=0.1453 0.0725 0.049
- link wsg_50_finger_left_link: geometry collision box size=0.0365 0.117 0.0122; visual mesh filename=package://schunk_description/meshes/wsg_50/finger_without_g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
- link wsg_50_finger_right_link: geometry collision box size=0.03 0.0344 0.0344; collision box size=0.0318 0.0318 0.037

File: software/models/common_components/schunk_description/urdf/wsg/wsg_50_no_gelsight_finger.urdf.xacro (robot description, xacro)
@@ -25,6 +25,4 @@
     </inertial>
     <!-- <xacro:left_finger_simple_visual/> -->
-    <xacro:left_finger_pretty_visual/>
-    <xacro:left_finger_simple_collision/>
   </link>
   <joint name="wsg_50_finger_right_joint" type="prismatic" >
@@ -41,7 +39,5 @@
       <inertia ixx="0.01" ixy="0" ixz="0" iyy="0.01" iyz="0" izz="0.01" />
     </inertial>
-    <!-- <xacro:right_finger_simple_visual/> -->
-    <xacro:right_finger_pretty_visual/>
-    <xacro:right_finger_simple_collision/>
+    <!-- no gelsight collision geometry -->
   </link>
   <!-- extensions -->
