Commit message: Replicated box pushing experiment well enough

File: software/models/IRB140/urdf/irb_140_ati_schunk_gelsight_one_finger.urdf.xacro (robot description, xacro)
@@ -1,8 +1,4 @@
 <?xml version="1.0" ?>
-<!-- =================================================================================== -->
-<!-- |    This document was autogenerated by xacro from irb_140_ati_schunk_gelsight_one_finger.urdf.xacro | -->
-<!-- |    EDITING THIS FILE BY HAND IS NOT RECOMMENDED                                 | -->
-<!-- =================================================================================== -->
-<robot name="IRB140" xmlns:xacro="http://www.ros.org/wiki/xacro">
+<robot name="IRB140" xmlns:xacro="http://ros.org/wiki/xacro">
   <link name="base_link">
     <inertial>
@@ -264,122 +260,5 @@
     <child link="ATI_sensor"/>
   </joint>
-  <!-- MATERIALS -->
-  <material name="Blue">
-    <color rgba="0 0 1 1"/>
-  </material>
-  <material name="Red">
-    <color rgba="1 0 0 1"/>
-  </material>
-  <material name="Green">
-    <color rgba="0 1 0 1"/>
-  </material>
-  <material name="Yellow">
-    <color rgba="1 1 0 1"/>
-  </material>
-  <material name="LightGrey">
-    <color rgba="0.6 0.6 0.6 1.0"/>
-  </material>
-  <!-- END OF MATERIALS -->
-  <!-- XACRO MACROS FOR VISUALS AND COLLISIONS -->
-  <!-- END OF XACRO MACROS -->
-  <link name="palm">
-    <inertial>
-      <origin rpy="0 0 0" xyz="0 0 0"/>
-      <mass value="1"/>
-      <inertia ixx="0.01" ixy="0" ixz="0" iyy="0.01" iyz="0" izz="0.01"/>
-    </inertial>
-    <visual>
-      <geometry>
-        <mesh filename="package://schunk_description/meshes/wsg_50/palm.stl"/>
-      </geometry>
-    </visual>
-    <!-- The gripper itself -->
-    <collision>
-      <geometry>
-        <box size="0.1453 0.0725 0.049"/>
-      </geometry>
-      <origin rpy="0 0 0" xyz="0.0 -0.0351 0.0"/>
-    </collision>
-    <!-- the larger mounting plate -->
-    <collision>
-      <geometry>
-        <box size="0.05 0.0064 0.095"/>
-      </geometry>
-      <origin rpy="0 0 0" xyz="0.0 0.007 0"/>
-    </collision>
-  </link>
-  <joint name="wsg_50_finger_left_joint" type="prismatic">
-    <origin rpy="0 1.5707 0" xyz="0 -0.0719 0"/>
-    <parent link="palm"/>
-    <child link="wsg_50_finger_left_link"/>
-    <axis xyz="0 0 -1"/>
-    <!--<limit effort="10" lower="-0.001" upper="0.109" velocity="1.0"/>-->
-  </joint>
-  <link name="wsg_50_finger_left_link">
-    <inertial>
-      <origin rpy="0 0 0" xyz="0 0 0"/>
-      <mass value="1"/>
-      <inertia ixx="0.01" ixy="0" ixz="0" iyy="0.01" iyz="0" izz="0.01"/>
-    </inertial>
-    <!-- <xacro:left_finger_pretty_visual/> -->
-  </link>
-  <joint name="wsg_50_finger_right_joint" type="prismatic">
-    <origin rpy="3.1415 -1.5707 0" xyz="0 -0.0719 0.0"/>
-    <parent link="palm"/>
-    <child link="wsg_50_finger_right_link"/>
-    <axis xyz="0 0 1"/>
-    <!--<limit effort="10" lower="-0.001" upper="0.109" velocity="1.0"/> -->
-  </joint>
-  <link name="wsg_50_finger_right_link">
-    <inertial>
-      <origin rpy="0 0 0" xyz="0 0 0"/>
-      <mass value="1"/>
-      <inertia ixx="0.01" ixy="0" ixz="0" iyy="0.01" iyz="0" izz="0.01"/>
-    </inertial>
-    <!-- <xacro:right_finger_pretty_visual/> -->
-    <visual>
-      <geometry>
-        <mesh filename="package://schunk_description/meshes/wsg_50/finger_with_gelsight.stl"/>
-      </geometry>
-    </visual>
-    <!-- Finger adapter and aluminum adapter block -->
-    <collision>
-      <geometry>
-        <box size="0.03 0.0344 0.0344"/>
-      </geometry>
-      <origin rpy="0 0 0" xyz="0.0 0.0172 0.0172"/>
-    </collision>
-    <!-- Stick to gelsight box and backplate / optotrak marker mount -->
-    <collision>
-      <geometry>
-        <box size="0.036 0.0883 0.0207"/>
-      </geometry>
-      <origin rpy="0 0 0" xyz="0.0 0.075 0.025"/>
-    </collision>
-    <!-- Gelsight box -->
-    <collision>
-      <geometry>
-        <box size="0.0318 0.0318 0.037"/>
-      </geometry>
-      <origin rpy="0 0 0" xyz="-0.0055 0.1005 0.01231"/>
-    </collision>
-  </link>
-  <!-- extensions -->
-  <transmission name="wsg_50_finger_left_trans">
-    <type>transmission_interface/SimpleTransmission</type>
-    <joint name="wsg_50_finger_left_joint"/>
-    <actuator name="wsg_50_finger_left_motor">
-      <hardwareInterface>EffortJointInterface</hardwareInterface>
-      <mechanicalReduction>1</mechanicalReduction>
-    </actuator>
-  </transmission>
-  <transmission name="wsg_50_finger_right_trans">
-    <type>transmission_interface/SimpleTransmission</type>
-    <joint name="wsg_50_finger_right_joint"/>
-    <actuator name="wsg_50_finger_right_motor">
-      <hardwareInterface>EffortJointInterface</hardwareInterface>
-      <mechanicalReduction>1</mechanicalReduction>
-    </actuator>
-  </transmission>
+  <xacro:include filename="$(find schunk_description)/urdf/wsg/wsg_50_one_finger.urdf.xacro" />
   <joint name="ati_joint" type="fixed">
     <origin rpy="3.1415 1.5707 0.0" xyz="0.0 0.073622 0.0"/>

File: software/models/common_components/schunk_description/urdf/wsg/wsg_50_no_gelsight_finger.urdf (robot description, URDF)
Before this commit: robot wsg_50, 3 links, 2 joints
Links:
- link wsg_50_finger_left_link: geometry 
- link wsg_50_finger_right_link: geometry 

File: software/models/common_components/schunk_description/urdf/wsg/wsg_50_one_finger.urdf (robot description, URDF)
Before this commit: robot wsg_50, 3 links, 2 joints
Links:
- link wsg_50_finger_right_link: geometry 

File: software/models/common_components/schunk_description/urdf/wsg/wsg_50_one_finger.urdf.xacro (robot description, xacro)
@@ -25,6 +25,4 @@
     </inertial>
     <!-- <xacro:left_finger_pretty_visual/> -->
-    <xacro:left_finger_pretty_visual/>
-    <xacro:left_finger_simple_collision/>
   </link>
   <joint name="wsg_50_finger_right_joint" type="prismatic" >
