Commit message: Nonpenetration and tinybolt tracking

File: software/models/IRB140/urdf/irb_140_ati_schunk_gelsight.urdf (robot description, URDF)
Before this commit: robot IRB140, 11 links, 9 joints
Links:
- link palm: geometry collision box size=0.05 0.0064 0.095; collision box size=0.1453 0.0725 0.049
- link wsg_50_finger_left_link: geometry collision box size=0.0365 0.117 0.0122; visual box size=0.0365 0.117 0.0122
- link wsg_50_finger_right_link: geometry collision box size=0.03 0.0344 0.0344; collision box size=0.0318 0.0318 0.037

File: software/models/common_components/schunk_description/urdf/wsg/visual_collisions.xacro (robot description, xacro)
@@ -79,8 +79,8 @@
   </xacro:macro>
   <xacro:macro name="left_finger_simple_visual" params="">
-    <xacro:visual_offset_box s_x="0.0365" s_y="0.117" s_z="0.0122" o_x="0.003" o_y="-0.0585" o_z="-0.0056"/>
+    <xacro:visual_offset_box s_x="0.0365" s_y="0.117" s_z="0.0122" o_x="0.003" o_y="-0.0585" o_z="-0.0106"/>
   </xacro:macro>
   <xacro:macro name="left_finger_simple_collision" params="">
-    <xacro:collision_offset_box s_x="0.0365" s_y="0.117" s_z="0.0122" o_x="0.003" o_y="-0.0585" o_z="-0.0056"/>
+    <xacro:collision_offset_box s_x="0.0365" s_y="0.117" s_z="0.0122" o_x="0.003" o_y="-0.0585" o_z="-0.0106"/>
   </xacro:macro>
   <xacro:macro name="right_finger_pretty_visual" params="">

File: software/models/common_components/schunk_description/urdf/wsg/wsg_50.urdf.xacro (robot description, xacro)
@@ -8,5 +8,5 @@
       <inertia ixx="0.01" ixy="0" ixz="0" iyy="0.01" iyz="0" izz="0.01" />
     </inertial>
-    <xacro:palm_pretty_visual/>
+    <xacro:palm_simple_visual/>
     <xacro:palm_simple_collision/>
   </link>
@@ -25,5 +25,5 @@
     </inertial>
     <!-- <xacro:left_finger_simple_visual/> -->
-    <xacro:left_finger_pretty_visual/>
+    <xacro:left_finger_simple_visual/>
     <xacro:left_finger_simple_collision/>
   </link>
@@ -42,5 +42,5 @@
     </inertial>
     <!-- <xacro:right_finger_simple_visual/> -->
-    <xacro:right_finger_pretty_visual/>
+    <xacro:right_finger_simple_visual/>
     <xacro:right_finger_simple_collision/>
   </link>

Commit message: log state for icra video

File: software/models/IRB140/urdf/irb_140_ati_schunk_gelsight.urdf (robot description, URDF)
Before this commit: robot IRB140, 11 links, 9 joints
Links:
- link wsg_50_finger_left_link: geometry collision box size=0.0365 0.117 0.0122; visual mesh filename=package://schunk_description/meshes/wsg_50/finger_without_g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
